File: kicad/BE511_Lab4_KiCadProject/BE511_Lab4_KiCadProject.kicad_sch (KiCad schematic)
At the start: 0 parts

Commit message: Complete schematic
Parts:
- added A1: Arduino_UNO_R3, Module:Arduino_UNO_R3, symbol MCU_Module:Arduino_UNO_R3
- added C1, C2, C3, C4: 3nF, symbol Device:C
- added C5, C6, C7: 0.1μF, symbol Device:C
- added J1, J4: Conn_02x05_Odd_Even, symbol Connector_Generic:Conn_02x05_Odd_Even
- added J2, J3: Screw_Terminal_01x05, symbol Connector:Screw_Terminal_01x05
- added R1, R2, R3, R4: 1k, symbol Device:R
- added U1: MCP3204, symbol Analog_ADC:MCP3204
- added U2, U3: MCP4922-EP, symbol Analog_DAC:MCP4922-EP
Connections:
- new net: C3.1, R3.1, U1.3 (CH2)
- new net: J1.6 (Pin_6), J2.3 (Pin_3), R3.2
- new net: C1.1, R1.1, U1.1 (CH0)
- new net: J3.1 (Pin_1), J4.1 (Pin_1), U2.14 (VoutA)
- new net: J3.2 (Pin_2), J4.3 (Pin_3), U2.10 (VoutB)
- new net: J3.3 (Pin_3), J4.5 (Pin_5), U3.14 (VoutA)
- new net: J3.4 (Pin_4), J4.7 (Pin_7), U3.10 (VoutB)
- new net: J1.2 (Pin_2), J2.1 (Pin_1), R1.2
- new net: C2.1, R2.1, U1.2 (CH1)
- new net: C4.1, R4.1, U1.4 (CH3)
- new net: J1.4 (Pin_4), J2.2 (Pin_2), R2.2
- new net: J1.8 (Pin_8), J2.4 (Pin_4), R4.2
- new net +5V: A1.5 (+5V), C5.1, C6.1, C7.1, U1.13 (Vref), U1.14 (Vdd), U2.1 (VDD), U2.11 (VrefB), U2.13 (VrefA), U3.1 (VDD), U3.11 (VrefB), U3.13 (VrefA)
- new net CIPO: A1.27 (D12), U1.10 (Dout)
- new net COPI: A1.26 (D11), U1.9 (Din), U2.5 (SDI), U3.5 (SDI)
- new net CS0: A1.25 (D10), U1.8 (~{CS}/SHDN)
- new net CS1: A1.24 (D9), U2.3 (~{CS})
- new net CS2: A1.23 (D8), U3.3 (~{CS})
- new net GND: A1.29 (GND), A1.6 (GND), A1.7 (GND), C1.2, C2.2, C3.2, C4.2, C5.2, C6.2, C7.2, J1.1 (Pin_1), J1.3 (Pin_3), J1.5 (Pin_5), J1.7 (Pin_7), J1.9 (Pin_9), J2.5 (Pin_5), J3.5 (Pin_5), J4.2 (Pin_2), J4.4 (Pin_4), J4.6 (Pin_6), J4.8 (Pin_8), U1.12 (AGND), U1.7 (DGND), U2.12 (AVSS), U3.12 (AVSS)
- new net SCK: A1.28 (D13), U1.11 (CLK), U2.4 (SCK), U3.4 (SCK)
- new net nLDAC: A1.22 (D7), U2.8 (~{LDAC}), U3.8 (~{LDAC})
- new net nSHDN: A1.21 (D6), U2.9 (~{SHDN}), U3.9 (~{SHDN})
- no-connect marks 0 -> 1

Commit message: Assign footprints, ERC clean
Parts:
- C1, C2, C3, C4, C5, C6, C7: footprint (none) -> Capacitor_THT:C_Disc_D4.7mm_W2.5mm_P5.00mm
- J1, J4: footprint (none) -> Connector_PinSocket_2.54mm:PinSocket_2x05_P2.54mm_Vertical
- J2, J3: footprint (none) -> TerminalBlock:TerminalBlock_Xinya_XY308-2.54-5P_1x05_P2.54mm_Horizontal
- R1, R2, R3, R4: footprint (none) -> Resistor_THT:R_Axial_DIN0207_L6.3mm_D2.5mm_P10.16mm_Horizontal
- U1, U2, U3: footprint (none) -> Package_DIP:DIP-14_W7.62mm
Changed lines of the file:
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@@
 			)
 		)
-		(property "Footprint" ""
+		(property "Footprint" "Resistor_THT:R_Axial_DIN0207_L6.3mm_D2.5mm_P10.16mm_Horizontal"
 			(at 72.39 61.722 90)
 			(hide yes)
@@
 			)
 		)
-		(property "Footprint" ""
+		(property "Footprint" "Capacitor_THT:C_Disc_D4.7mm_W2.5mm_P5.00mm"
 			(at 80.9752 85.09 0)
 			(hide yes)
@@
 			)
 		)
-		(property "Footprint" ""
+		(property "Footprint" "TerminalBlock:TerminalBlock_Xinya_XY308-2.54-5P_1x05_P2.54mm_Horizontal"
 			(at 259.08 60.96 0)
 			(hide yes)
@@
 			)
 		)
-		(property "Footprint" ""
+		(property "Footprint" "Resistor_THT:R_Axial_DIN0207_L6.3mm_D2.5mm_P10.16mm_Horizontal"
 			(at 72.39 54.102 90)
 			(hide yes)
@@
 			)
 		)
-		(property "Footprint" ""
+		(property "Footprint" "Connector_PinSocket_2.54mm:PinSocket_2x05_P2.54mm_Vertical"
 			(at 259.08 92.71 0)
 			(hide yes)
@@
 			)
 		)
-		(property "Footprint" ""
+		(property "Footprint" "Package_DIP:DIP-14_W7.62mm"
 			(at 139.7 68.58 0)
 			(hide yes)
@@
 			)
 		)
-		(property "Footprint" ""
+		(property "Footprint" "Package_DIP:DIP-14_W7.62mm"
 			(at 191.77 60.96 0)
 			(hide yes)
@@
 			)
 		)
-		(property "Footprint" ""
+		(property "Footprint" "Capacitor_THT:C_Disc_D4.7mm_W2.5mm_P5.00mm"
 			(at 167.3352 95.25 0)
 			(hide yes)
@@
 			)
 		)
-		(property "Footprint" ""
+		(property "Footprint" "Capacitor_THT:C_Disc_D4.7mm_W2.5mm_P5.00mm"
 			(at 100.0252 85.09 0)
 			(hide yes)
@@
 			)
 		)
-		(property "Footprint" ""
+		(property "Footprint" "Connector_PinSocket_2.54mm:PinSocket_2x05_P2.54mm_Vertical"
 			(at 40.64 93.98 0)
 			(hide yes)
@@
 			)
 		)
-		(property "Footprint" ""
+		(property "Footprint" "Resistor_THT:R_Axial_DIN0207_L6.3mm_D2.5mm_P10.16mm_Horizontal"
 			(at 72.39 65.532 90)
 			(hide yes)
@@
 			)
 		)
-		(property "Footprint" ""
+		(property "Footprint" "Resistor_THT:R_Axial_DIN0207_L6.3mm_D2.5mm_P10.16mm_Horizontal"
 			(at 72.39 57.912 90)
 			(hide yes)
@@
 			)
 		)
-		(property "Footprint" ""
+		(property "Footprint" "Capacitor_THT:C_Disc_D4.7mm_W2.5mm_P5.00mm"
 			(at 172.4152 36.83 0)
 			(hide yes)
@@
 			)
 		)
-		(property "Footprint" ""
+		(property "Footprint" "TerminalBlock:TerminalBlock_Xinya_XY308-2.54-5P_1x05_P2.54mm_Horizontal"
 			(at 36.83 62.23 0)
 			(hide yes)
@@
 			)
 		)
-		(property "Footprint" ""
+		(property "Footprint" "Package_DIP:DIP-14_W7.62mm"
 			(at 191.77 110.49 0)
 			(hide yes)
@@
 			)
 		)
-		(property "Footprint" ""
+		(property "Footprint" "Capacitor_THT:C_Disc_D4.7mm_W2.5mm_P5.00mm"
 			(at 93.6752 85.09 0)
 			(hide yes)
@@
 			)
 		)
-		(property "Footprint" ""
+		(property "Footprint" "Capacitor_THT:C_Disc_D4.7mm_W2.5mm_P5.00mm"
 			(at 87.3252 85.09 0)
 			(hide yes)
@@
 			)
 		)
-		(property "Footprint" ""
+		(property "Footprint" "Capacitor_THT:C_Disc_D4.7mm_W2.5mm_P5.00mm"
 			(at 102.5652 40.64 0)
 			(hide yes)
